Commit message: commented map

File: src/pioneer3at_ros/urdf/pioneer3at_ros.urdf (robot description, URDF)
Before this commit: robot robot, 7 links, 6 joints
Links:
- link base_link: geometry collision box size=0.501 0.300 0.19; visual mesh filename=package://pioneer3at_ros/meshes/chassis.dae scale=1.0 1.0 1.0
- link left_front_wheel: geometry collision cylinder length=0.075 radius=0.110; visual mesh filename=package://pioneer3at_ros/meshes/wheel.dae scale=1.0 1.0 1.0
- link left_rear_wheel: geometry collision cylinder length=0.075 radius=0.110; visual mesh filename=package://pioneer3at_ros/meshes/wheel.dae scale=1.0 1.0 1.0
- link right_front_wheel: geometry collision cylinder length=0.075 radius=0.110; visual mesh filename=package://pioneer3at_ros/meshes/wheel.dae scale=1.0 1.0 1.0
- link right_rear_wheel: geometry collision cylinder length=0.075 radius=0.110; visual mesh filename=package://pioneer3at_ros/meshes/wheel.dae scale=1.0 1.0 1.0
