Commit message: first map

File: src/pioneer3at/pioneer3at_description/urdf/pioneer3at_ros.urdf (robot description, URDF)
Before this commit: robot robot, 7 links, 6 joints
Joints:
- joint camera_joint: origin xyz=0.1   0    0.45 rpy=0  0  0 -> xyz=0.1   0    0.40 rpy=0  0  0
- joint hokuyo_joint: origin xyz=0.1   0    0.35 rpy=0  0  0 -> xyz=0.1   0    0.315 rpy=0  0  0

Commit message: rtabmap working

File: src/pioneer3at/pioneer3at_description/urdf/pioneer3at_ros.urdf (robot description, URDF)
Before this commit: robot robot, 7 links, 6 joints
Joints:
- joint camera_joint: origin xyz=0.1   0    0.40 rpy=0  0  0 -> xyz=0.1   0    0.40 rpy=0  0 0
