Commit message: p3at teleoperation and drone rtabmap

File: src/pioneer3at/pioneer3at_description/urdf/pioneer3at_depth_ros.urdf (robot description, URDF)
Before this commit: robot robot, 7 links, 6 joints
Links:
- link camera_link: geometry collision box size=0.073 0.276 0.072; collision box size=0.1 0.1 0.07
Joints:
- joint camera_joint: origin xyz=0.1   0    0.33 rpy=0  0  0 -> xyz=0.1   0    0.37 rpy=0  0.08  0
