Commit message: UAV camera new angle

File: src/quadrotor/hector_moveit/hector_quadrotor/hector_quadrotor_description/urdf/quadrotor_with_kinect.urdf.xacro (robot description, xacro)
@@ -9,5 +9,5 @@
     <xacro:include filename="$(find hector_sensors_description)/urdf/kinect_camera.urdf.xacro" />
     <xacro:kinect_camera name="camera" parent="base_link">
-      <origin xyz="0.23 0.0 -0.1" rpy="0 0 0"/>
+      <origin xyz="0.13 0.0 -0.1" rpy="0 0.262 0"/>
     </xacro:kinect_camera>
 </robot>
